Commit message: Reconstucture something

File: urdf/my_robot.urdf (robot description, URDF)
Before this commit: robot test_robot, 4 links, 3 joints
Joints:
- joint joint1: origin xyz=5 3 0 rpy=0 0 0 -> xyz=5 0.6 0 rpy=0 0 0
- joint joint2: origin xyz=-2 5 0 rpy=0 0 1.57 -> xyz=-0.4 1 0 rpy=0 0 1.57
- joint joint3: origin xyz=5 0 0 rpy=0 0 -1.57 -> xyz=1 0 0 rpy=0 0 -1.57

File: urdf/one_shape.urdf (robot description, URDF)
Before this commit: robot myfirst, 1 links, 0 joints
Links:
- removed link base_link
- added link camera; visual cylinder length=0.6 radius=0.2
