Commit message: Edit can use

File: urdf/real_cage.urdf (robot description, URDF)
Before this commit: robot cage, 14 links, 13 joints
Links:
- link base_cage: geometry visual cylinder length=2 radius=0.1
- link base_cage_back: geometry visual cylinder length=2 radius=0.1
- link base_cage_back_bottom: geometry visual cylinder length=2 radius=0.1
- link base_cage_back_left: geometry visual cylinder length=1 radius=0.1
- link base_cage_back_right: geometry visual cylinder length=1 radius=0.1
- link base_cage_beside_left_bottom: geometry visual cylinder length=2 radius=0.1
- link base_cage_beside_left_top: geometry visual cylinder length=2 radius=0.1
- link base_cage_beside_right_bottom: geometry visual cylinder length=2 radius=0.1
- link base_cage_beside_right_top: geometry visual cylinder length=2 radius=0.1
- link base_cage_front_bottom: geometry visual cylinder length=2 radius=0.1
- link base_cage_front_left: geometry visual cylinder length=1 radius=0.1
- link base_cage_front_right: geometry visual cylinder length=1 radius=0.1

Commit message: Abort to write cpp

File: urdf/real_cage.urdf (robot description, URDF)
Before this commit: robot cage, 14 links, 13 joints
Links:
- link base_cage: geometry visual cylinder length=2 radius=${radius_of_cylinder}
- link base_cage_back: geometry visual cylinder length=2 radius=${radius_of_cyliner}
- link base_cage_back_bottom: geometry visual cylinder length=2 radius=${radius_of_cyliner}
- link base_cage_back_left: geometry visual cylinder length=1 radius=${radius_of_cyliner}
- link base_cage_back_right: geometry visual cylinder length=1 radius=${radius_of_cyliner}
- link base_cage_beside_left_bottom: geometry visual cylinder length=2 radius=${radius_of_cyliner}
- link base_cage_beside_left_top: geometry visual cylinder length=2 radius=${radius_of_cyliner}
- link base_cage_beside_right_bottom: geometry visual cylinder length=2 radius=${radius_of_cyliner}
- link base_cage_beside_right_top: geometry visual cylinder length=2 radius=${radius_of_cyliner}
- link base_cage_front_bottom: geometry visual cylinder length=2 radius=${radius_of_cyliner}
- link base_cage_front_left: geometry visual cylinder length=1 radius=${radius_of_cyliner}
- link base_cage_front_right: geometry visual cylinder length=1 radius=${radius_of_cyliner}

Commit message: Use xacro and finish about bag

File: urdf/real_cage.urdf (robot description, URDF)
Before this commit: robot cage, 14 links, 13 joints
Links:
- link base_cage_back: geometry visual cylinder length=2 radius=${radius_of_cylinder}
- link base_cage_back_bottom: geometry visual cylinder length=2 radius=${radius_of_cylinder}
- link base_cage_back_left: geometry visual cylinder length=1 radius=${radius_of_cylinder}
- link base_cage_back_right: geometry visual cylinder length=1 radius=${radius_of_cylinder}
- link base_cage_beside_left_bottom: geometry visual cylinder length=2 radius=${radius_of_cylinder}
- link base_cage_beside_left_top: geometry visual cylinder length=2 radius=${radius_of_cylinder}
- link base_cage_beside_right_bottom: geometry visual cylinder length=2 radius=${radius_of_cylinder}
- link base_cage_beside_right_top: geometry visual cylinder length=2 radius=${radius_of_cylinder}
- link base_cage_front_bottom: geometry visual cylinder length=2 radius=${radius_of_cylinder}
- link base_cage_front_left: geometry visual cylinder length=1 radius=${radius_of_cylinder}
- link base_cage_front_right: geometry visual cylinder length=1 radius=${radius_of_cylinder}
